File: SerialToUsb/S2U_Daughter.brd (EAGLE design)
At the start: 30.5 x 12.7 mm, 1 part

Commit message: some changes
Parts:
- added U$2: CH340, S2U_lib:SSOP20
- added U$3: MAX3241E, S2U_lib:TSSOP28
- moved U$1 13.4 mm to (14.6, -6.99)
Connections:
- new net N$1: U$1.GND, U$1.GND$1
- new net N$2: U$1.VCC
Changed lines of the file:
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@@
 </autorouter>
 <elements>
-<element name="U$1" library="S2U_lib" package="S2U_DAUGHTER_HEADERS" value="S2U_DAUGHTER" x="13.97" y="6.35"/>
+<element name="U$1" library="S2U_lib" package="S2U_DAUGHTER_HEADERS" value="S2U_DAUGHTER" x="14.605" y="-6.985"/>
+<element name="U$2" library="S2U_lib" package="SSOP20" value="CH340" x="6.35" y="-18.415"/>
+<element name="U$3" library="S2U_lib" package="TSSOP28" value="MAX3241E" x="6.985" y="-26.67"/>
 </elements>
 <signals>
+<signal name="N$1">
+<contactref element="U$1" pad="GND"/>
+<contactref element="U$1" pad="GND$1"/>
+<wire x1="3.175" y1="-10.795" x2="23.495" y2="-8.255" width="0" layer="19" extent="1-1"/>
+</signal>
+<signal name="N$2">
+<contactref element="U$1" pad="VCC"/>
+</signal>
 </signals>
 </board>
