File: SerialToUsb/S2U_Daughter.sch (EAGLE design)
At the start: 1 part

Commit message: some changes
Parts:
- added U$2: CH340, S2U_lib:CH340
- added U$3: MAX3241E, S2U_lib:MAX3241E
Connections:
- new net N$1: U$1.GND$1, U$1.GND$2
- new net N$2: U$1.VCC
Changed lines of the file:
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@@
 <parts>
 <part name="U$1" library="S2U_lib" deviceset="S2U_DAUGHTER" device=""/>
+<part name="U$2" library="S2U_lib" deviceset="CH340" device=""/>
+<part name="U$3" library="S2U_lib" deviceset="MAX3241E" device=""/>
 </parts>
 <sheets>
@@
 </plain>
 <instances>
-<instance part="U$1" gate="G$1" x="71.12" y="50.8"/>
+<instance part="U$1" gate="G$1" x="71.12" y="48.26"/>
+<instance part="U$2" gate="G$1" x="76.2" y="12.7"/>
+<instance part="U$3" gate="G$1" x="116.84" y="38.1"/>
 </instances>
 <busses>
 </busses>
 <nets>
+<net name="N$1" class="0">
+<segment>
+<pinref part="U$1" gate="G$1" pin="GND$1"/>
+<wire x1="55.88" y1="45.72" x2="53.34" y2="45.72" width="0.1524" layer="91"/>
+<wire x1="53.34" y1="45.72" x2="53.34" y2="43.18" width="0.1524" layer="91"/>
+<pinref part="U$1" gate="G$1" pin="GND$2"/>
+<wire x1="53.34" y1="43.18" x2="55.88" y2="43.18" width="0.1524" layer="91"/>
+<wire x1="53.34" y1="43.18" x2="53.34" y2="38.1" width="0.1524" layer="91"/>
+<junction x="53.34" y="43.18"/>
+</segment>
+</net>
+<net name="N$2" class="0">
+<segment>
+<pinref part="U$1" gate="G$1" pin="VCC"/>
+<wire x1="55.88" y1="58.42" x2="53.34" y2="58.42" width="0.1524" layer="91"/>
+<wire x1="53.34" y1="58.42" x2="53.34" y2="60.96" width="0.1524" layer="91"/>
+</segment>
+</net>
 </nets>
 </sheet>
